File: _autosave-SoftwareDebugPicoHat.kicad_pcb (KiCad board)
At the start: 4 copper layers, 69 x 54.7 mm, 13 parts, among them J1 35362-0950, J2 Conn_Coaxial, J3 USB_C_Receptacle_USB2.0_14P, J4 Conn_Coaxial, J5 Conn_01x04_Pin, U1 RFM98PW, U3 LORA1280F27-TCXO

Commit message: Fixed Scem
Connections:
- U3 pad 2: SBAND_TCXOEN -> +3V3
Routing:
- net SBAND_TCXOEN: track 3.22 -> 0.00 mm
- net +3V3: track 119.5 -> 122.2 mm
- net +5V: track 149.4 -> 150.2 mm
- net GND: vias 132 -> 133
